File: MainBoard.sch (KiCad schematic (older format))
At the start: 15 parts, among them P1 CARTRIDGE_SLOT, P2 FRONT_PANEL_CONNECTOR, U1 S-CPU, U13 S-SMP, U14 S-DSP, U15 PSRAM, U16 PSRAM, U17 UPD6376, U2 S-PPU1, U3 S-PPU2, U4 SRAM, U5 SRAM, U6 S-WRAM, U8 CIC, U9 74AHC04

Commit message: Replaced with local copy footprints
Parts:
- P1: footprint (none) -> SNES:SNES_RETRODE_SLOT
- U1, U2, U3: footprint Package_QFP:PQFP-100_14x20mm_P0.65mm -> SNES:PQFP-100_14x20mm_P0.65mm
- U14: footprint Package_QFP:PQFP-80_14x20mm_P0.8mm -> SNES:PQFP-80_14x20mm_P0.8mm
- U16, U4, U5: footprint Package_SO:SSOP-28_5.3x10.2mm_P0.65mm -> SNES:SSOP-28_5.3x10.2mm_P0.65mm
- U17: footprint Package_SO:SOIC-16W_5.3x10.2mm_P1.27mm -> SNES:SOIC-16W_5.3x10.2mm_P1.27mm
- U8: footprint Package_SO:SSOP-18_4.4x6.5mm_P0.65mm -> SNES:SSOP-18_4.4x6.5mm_P0.65mm
Other:
- moved on the sheet: U16
Changed lines of the file:
@@
 F 0 "U1" H 2900 4450 50  0000 C CNN
 F 1 "S-CPU" H 2900 -850 50  0000 C CNN
-F 2 "Package_QFP:PQFP-100_14x20mm_P0.65mm" H 2900 4450 50  0001 C CNN
+F 2 "SNES:PQFP-100_14x20mm_P0.65mm" H 2900 4450 50  0001 C CNN
 F 3 "" H 2900 4450 50  0001 C CNN
 	1    2900 4450
@@
 F 0 "U2" H 6350 4450 50  0000 C CNN
 F 1 "S-PPU1" H 6350 -850 50  0000 C CNN
-F 2 "Package_QFP:PQFP-100_14x20mm_P0.65mm" H 6350 4450 50  0001 C CNN
+F 2 "SNES:PQFP-100_14x20mm_P0.65mm" H 6350 4450 50  0001 C CNN
 F 3 "" H 6350 4450 50  0001 C CNN
 	1    6350 4450
@@
 F 0 "U3" H 12350 4450 50  0000 C CNN
 F 1 "S-PPU2" H 12350 -850 50  0000 C CNN
-F 2 "Package_QFP:PQFP-100_14x20mm_P0.65mm" H 12350 4450 50  0001 C CNN
+F 2 "SNES:PQFP-100_14x20mm_P0.65mm" H 12350 4450 50  0001 C CNN
 F 3 "" H 12350 4450 50  0001 C CNN
 	1    12350 4450
@@
 F 0 "U4" H 8250 4450 50  0000 C CNN
 F 1 "SRAM" H 8250 2750 50  0000 C CNN
-F 2 "Package_SO:SSOP-28_5.3x10.2mm_P0.65mm" H 8250 4350 50  0001 C CNN
+F 2 "SNES:SSOP-28_5.3x10.2mm_P0.65mm" H 8250 4350 50  0001 C CNN
 F 3 "" H 8250 4350 50  0001 C CNN
 	1    8250 4450
@@
 F 0 "U5" H 8250 6950 50  0000 C CNN
 F 1 "SRAM" H 8250 5250 50  0000 C CNN
-F 2 "Package_SO:SSOP-28_5.3x10.2mm_P0.65mm" H 8250 6850 50  0001 C CNN
+F 2 "SNES:SSOP-28_5.3x10.2mm_P0.65mm" H 8250 6850 50  0001 C CNN
 F 3 "" H 8250 6850 50  0001 C CNN
 	1    8250 6950
@@
 U 1 1 5FE7850A
 P 7450 11450
-F 0 "P1" H 7450 11575 50  0000 C CNN
-F 1 "CARTRIDGE_SLOT" H 7450 11484 50  0000 C CNN
-F 2 "" H 7450 11450 50  0001 C CNN
+F 0 "P1" H 7450 11450 50  0000 C CNN
+F 1 "CARTRIDGE_SLOT" H 7450 8250 50  0000 C CNN
+F 2 "SNES:SNES_RETRODE_SLOT" H 7450 11450 50  0001 C CNN
 F 3 "" H 7450 11450 50  0001 C CNN
 	1    7450 11450
@@
 U 1 1 5FE7DEEB
 P 3800 15950
-F 0 "U8" H 3800 16075 50  0000 C CNN
-F 1 "CIC" H 3800 15984 50  0000 C CNN
-F 2 "Package_SO:SSOP-18_4.4x6.5mm_P0.65mm" H 3800 15950 50  0001 C CNN
+F 0 "U8" H 3800 15950 50  0000 C CNN
+F 1 "CIC" H 3800 14950 50  0000 C CNN
+F 2 "SNES:SSOP-18_4.4x6.5mm_P0.65mm" H 3800 15950 50  0001 C CNN
 F 3 "" H 3800 15950 50  0001 C CNN
 	1    3800 15950
@@
 U 1 1 5FE7F002
 P 6800 16500
-F 0 "U9" H 6800 16817 50  0000 C CNN
-F 1 "74AHC04" H 6800 16726 50  0000 C CNN
+F 0 "U9" H 6800 16650 50  0000 C CNN
+F 1 "74AHC04" H 6800 16300 50  0000 C CNN
 F 2 "" H 6800 16500 50  0001 C CNN
 F 3 "https://assets.nexperia.com/documents/data-sheet/74AHC_AHCT04.pdf" H 6800 16500 50  0001 C CNN
@@
 U 1 1 5FE85522
 P 12300 13950
-F 0 "U13" H 12300 14075 50  0000 C CNN
-F 1 "S-SMP" H 12300 13984 50  0000 C CNN
+F 0 "U13" H 12300 13950 50  0000 C CNN
+F 1 "S-SMP" H 12300 10650 50  0000 C CNN
 F 2 "" H 12300 13950 50  0001 C CNN
 F 3 "" H 12300 13950 50  0001 C CNN
@@
 U 1 1 5FE878B4
 P 14800 13950
-F 0 "U14" H 14800 14075 50  0000 C CNN
-F 1 "S-DSP" H 14800 13984 50  0000 C CNN
-F 2 "Package_QFP:PQFP-80_14x20mm_P0.8mm" H 14800 13950 50  0001 C CNN
+F 0 "U14" H 14800 13950 50  0000 C CNN
+F 1 "S-DSP" H 14800 9850 50  0000 C CNN
+F 2 "SNES:PQFP-80_14x20mm_P0.8mm" H 14800 13950 50  0001 C CNN
 F 3 "" H 14800 13950 50  0001 C CNN
 	1    14800 13950
@@
 U 1 1 5FE89DF5
 P 16750 13950
-F 0 "U15" H 16750 14075 50  0000 C CNN
-F 1 "PSRAM" H 16750 13984 50  0000 C CNN
+F 0 "U15" H 16750 13950 50  0000 C CNN
+F 1 "PSRAM" H 16750 12250 50  0000 C CNN
 F 2 "Package_SO:SSOP-28_5.3x10.2mm_P0.65mm" H 16750 13850 50  0001 C CNN
 F 3 "" H 16750 13850 50  0001 C CNN
@@
 L SNES:PSRAM U16
 U 1 1 5FE8B345
-P 16550 16290
-F 0 "U16" H 16550 16415 50  0000 C CNN
-F 1 "PSRAM" H 16550 16324 50  0000 C CNN
-F 2 "Package_SO:SSOP-28_5.3x10.2mm_P0.65mm" H 16550 16190 50  0001 C CNN
-F 3 "" H 16550 16190 50  0001 C CNN
-	1    16550 16290
+P 16750 16450
+F 0 "U16" H 16750 16450 50  0000 C CNN
+F 1 "PSRAM" H 16750 14750 50  0000 C CNN
+F 2 "SNES:SSOP-28_5.3x10.2mm_P0.65mm" H 16750 16350 50  0001 C CNN
+F 3 "" H 16750 16350 50  0001 C CNN
+	1    16750 16450
 	1    0    0    -1
 $EndComp
@@
 F 0 "U17" H 14750 11450 50  0000 C CNN
 F 1 "UPD6376" H 14750 10550 50  0000 C CNN
-F 2 "Package_SO:SOIC-16W_5.3x10.2mm_P1.27mm" H 14800 11450 50  0001 C CNN
+F 2 "SNES:SOIC-16W_5.3x10.2mm_P1.27mm" H 14800 11450 50  0001 C CNN
 F 3 "https://cdn.datasheetspdf.com/pdf-down/U/P/D/UPD6376_NEC.pdf" H 14800 11450 50  0001 C CNN
 	1    14750 11450
@@
 U 2 1 5FE96E9B
 P 6200 17000
-F 0 "U9" H 6200 17317 50  0000 C CNN
-F 1 "74AHC04" H 6200 17226 50  0000 C CNN
+F 0 "U9" H 6200 16850 50  0000 C CNN
+F 1 "74AHC04" H 6200 17200 50  0000 C CNN
 F 2 "" H 6200 17000 50  0001 C CNN
 F 3 "https://assets.nexperia.com/documents/data-sheet/74AHC_AHCT04.pdf" H 6200 17000 50  0001 C CNN

Commit message: JPIO port wired
Parts:
- added C107: 0.01uF, symbol Device:C_Small
- added C35, C36, C37, C38, C39, C40, C41, C42, C43: 330pF, symbol Device:C_Small
- added DA109, DA87, DA? (x3): BAT54C, Package_TO_SOT_SMD:SOT-23, symbol Diode:BAT54C
- added DA32, DA54, DA? (x3): BAT54A, Package_TO_SOT_SMD:SOT-23, symbol Diode:BAT54A
- added RN7882, RN?: 10K, Resistor_SMD:R_Array_Convex_4x0603, symbol Device:R_Pack04
- added RN8391: 100, symbol Device:R_Pack05
- added RN8490: 100, Resistor_SMD:R_Array_Convex_4x0603, symbol Device:R_Pack04
- U6: footprint (none) -> SNES:SOP-64_10.8x28mm_P0.8mm
Connections:
- net labels added: 4016.D0, 4016.D2, 4017.D0, 4017.D1, GND, JPCLK1, JPCLK2, JPIO6, JPIO7, JPSTR, VCC
- wire segments 0 -> 157
- no-connect marks 2 -> 6

Commit message: S-CPU started
Parts:
- added C90: 0.1uF, symbol Device:C_Small
- P2: symbol SNES:FRONT_PANEL_CONNECTOR -> SNES:FRONT_PANEL
- gave numbers to parts that had none: 6
- renumbered DA109 to DA10, DA32 to DA4, DA54 to DA5, DA87 to DA9
Connections:
- net labels added: 4016.D1, Post_Amplifier
- wire segments 157 -> 212
- no-connect marks 6 -> 24

Commit message: S-PPU1 + VRAM1
Parts:
- added C31: 0.01uF 50V, symbol Device:C_Small
- added C67: 1000uF 25V, symbol Device:CP_Small
- added C91, C93: 0.1uF, symbol Device:C_Small
- added D1: PB1100, Diode_SMD:D_SMA, symbol Device:D_Schottky_Small
- added F1: Polyfuse, Fuse:Fuse_1812_4532Metric, symbol Device:Polyfuse_Small
- added J1: USB B Mini, symbol Connector:USB_B_Mini
- added R92: 10K, Resistor_SMD:R_0603_1608Metric, symbol Device:R_Small
Connections:
- net labels added: CA0, CA1, CA10, CA11, CA12, CA13, CA14, CA15, CA16, CA17, CA18, CA19, CA2, CA20, CA21, CA22, CA23, CA3, CA4, CA5, CA6, CA7, CA8, CA9, CA[0..23], ~CPURD, ~CPURW, ~PARD, ~PAWR, ~RAMSEL, ~ROMSEL
- wire segments 212 -> 305
- no-connect marks 24 -> 28
Other:
- note added: "DC Power Input\nUSB +5V @ 1.7A\nDerived from +10V @ 0.85A"

Commit message: VRAM1 + VRAM2 + S-PPU1
Parts:
- added C94: 0.1uF, symbol Device:C_Small
Connections:
- net labels added: VA14, VAA0, VAA1, VAA10, VAA11, VAA12, VAA13, VAA2, VAA3, VAA4, VAA5, VAA6, VAA7, VAA8, VAA9, VAB0, VAB1, VAB10, VAB11, VAB12, VAB13, VAB2, VAB3, VAB4, VAB5, VAB6, VAB7, VAB8, VAB9, VDA0, VDA1, VDA2, VDA3, VDA4, VDA5, VDA6, VDA7, VDB0, VDB1, VDB2, VDB3, VDB4, VDB5, VDB6, VDB7, ~VARW, ~VBRW, ~VRD
- wire segments 305 -> 427

Commit message: VRAM rd/wr bus finished
Parts:
- gave numbers to parts that had none: 1
Connections:
- net labels added: ~VAWR, ~VBWR
- wire segments 427 -> 431

Commit message: Cart slot and PPU somewhat wired up
Parts:
- added C95: 0.1uF, symbol Device:C_Small
- added RA1: 100, Resistor_SMD:R_0603_1608Metric, symbol Device:R_Small
Connections:
- net labels added: D0, D1, D2, D3, D4, D5, D6, D7, PA0, PA1, PA2, PA3, PA4, PA5, PA6, PA7, ~CPUWR
- net labels removed: CA[0..23], ~CPURW, ~VARW, ~VBRW
- wire segments 431 -> 596
- no-connect marks 28 -> 27
Other:
- moved on the sheet: P1

Commit message: S-PPU2 wiring started
Parts:
- added C92: 0.1uF, symbol Device:C_Small
Connections:
- net labels added: CHR0, CHR1, CHR2, CHR3, COLOR0, COLOR1, COLOR2, FIELD, PRIO0, PRIO1, ~5MIN, ~HCLD, ~OVER, ~VCLD
- wire segments 596 -> 660
- no-connect marks 27 -> 40
Other:
- note added: "Consider employing DCP\nsuch as TPS2513"
