File: MainBoard.sch (KiCad schematic (older format))
At the start: 52 parts, among them J1 USB B Mini, P1 CARTRIDGE_SLOT, P2 FRONT_PANEL_CONNECTOR, U1 S-CPU, U13 S-SMP, U14 S-DSP, U15 PSRAM, U16 PSRAM, U17 UPD6376, U2 S-PPU1, U3 S-PPU2, U4 SRAM, U5 SRAM, U6 S-WRAM, U8 CIC, U9 74AHC04

Commit message: CIC completed, Xtal started
Parts:
- added C29: 0.1uF, symbol Device:C_Small
- added C62: 2.2uF, symbol Device:CP_Small
- added C70: 82pF, symbol Device:C_Small
- added SW1: RESET, Button_Switch_SMD:SW_Push_SPST_NO_Alps_SKRK, symbol Switch:SW_Push
- added unit 3 of U9
- added unit 4 of U9
- added unit 6 of U9
- added unit 5 of U9
- U9: value 74AHC04 -> HCU04
Connections:
- net labels added: CIC0, CIC1, CIC2, CIC3, IRQ, SCLK, ~RESET
- wire segments 660 -> 762
- no-connect marks 40 -> 50
Other:
- moved on the sheet: P1, U13, U14, U6, U8

Commit message: U11 added
Parts:
- added C89: 100nF, symbol Device:C_Small
- added R75: 100K, symbol Device:R_Small
- added U11: PST529D, symbol SNES:PST529D
- P2: footprint (none) -> SNES:SNES_JOYPAD_PORT_ZIP-11
Connections:
- wire segments 762 -> 777
Other:
- note added: "Power Supervisor\nMMP-3A package"
Changed lines of the file:
@@
 F 0 "P2" H 5900 2200 50  0000 C CNN
 F 1 "FRONT_PANEL_CONNECTOR" H 5900 2100 50  0000 C CNN
-F 2 "" H 5800 2100 50  0001 C CNN
+F 2 "SNES:SNES_JOYPAD_PORT_ZIP-11" H 5800 2100 50  0001 C CNN
 F 3 "" H 5800 2100 50  0001 C CNN
 	1    5900 2100
@@
 ~RESET
 Wire Wire Line
-	11600 2250 11600 5350
+	11600 3100 11600 5350
 Wire Wire Line
 	11600 5350 11900 5350
@@
 Wire Wire Line
 	14200 2800 14100 2800
+Connection ~ 14200 3250
+Entry Wire Line
+	9500 3900 9600 4000
+Wire Wire Line
+	9600 4000 10500 4000
+Wire Wire Line
+	10500 4000 10500 7550
+Wire Wire Line
+	10500 7550 11900 7550
+Text Label 9700 4000 0    50   ~ 0
+JPIO7
+Text Label 10600 7550 0    50   ~ 0
+JPIO7
+$Comp
+L SNES:PST529D U11
+U 1 1 601156A9
+P 12100 2950
+F 0 "U11" H 11800 2950 50  0000 L CNN
+F 1 "PST529D" H 12400 2950 50  0000 R CNN
+F 2 "" H 12100 2950 50  0001 C CNN
+F 3 "https://www.digchip.com/datasheets/download_datasheet.php?id=1395437&part-number=PST529" H 12100 2950 50  0001 C CNN
+	1    12100 2950
+	1    0    0    -1
+$EndComp
+Wire Wire Line
+	11700 3100 11600 3100
+$Comp
+L power:VCC #PWR?
+U 1 1 604448C6
+P 11600 2600
+F 0 "#PWR?" H 11600 2450 50  0001 C CNN
+F 1 "VCC" H 11615 2773 50  0000 C CNN
+F 2 "" H 11600 2600 50  0001 C CNN
+F 3 "" H 11600 2600 50  0001 C CNN
+	1    11600 2600
+	1    0    0    -1
+$EndComp
+$Comp
+L Device:R_Small R75
+U 1 1 604458D2
+P 11600 2900
+F 0 "R75" H 11542 2854 50  0000 R CNN
+F 1 "100K" H 11542 2945 50  0000 R CNN
+F 2 "" H 11600 2900 50  0001 C CNN
+F 3 "~" H 11600 2900 50  0001 C CNN
+	1    11600 2900
+	1    0    0    1
+$EndComp
+Wire Wire Line
+	11600 3000 11600 3100
+Connection ~ 11600 3100
+Wire Wire Line
+	11600 2800 11600 2700
+Wire Wire Line
+	11600 2700 12600 2700
+Wire Wire Line
+	12600 2700 12600 3100
+Wire Wire Line
+	12600 3100 12500 3100
+Connection ~ 11600 2700
+Wire Wire Line
+	11600 2700 11600 2600
+$Comp
+L Device:C_Small C89
+U 1 1 6119D252
+P 12600 3300
+F 0 "C89" H 12692 3346 50  0000 L CNN
+F 1 "100nF" H 12692 3255 50  0000 L CNN
+F 2 "" H 12600 3300 50  0001 C CNN
+F 3 "~" H 12600 3300 50  0001 C CNN
+	1    12600 3300
+	1    0    0    -1
+$EndComp
+$Comp
+L power:GND #PWR?
+U 1 1 6037A7EC
+P 12100 3700
+F 0 "#PWR?" H 12100 3450 50  0001 C CNN
+F 1 "GND" H 12105 3527 50  0000 C CNN
+F 2 "" H 12100 3700 50  0001 C CNN
+F 3 "" H 12100 3700 50  0001 C CNN
+	1    12100 3700
+	1    0    0    -1
+$EndComp
+Wire Wire Line
+	12100 3500 12100 3600
+Wire Wire Line
+	12600 3400 12600 3600
+Wire Wire Line
+	12600 3600 12100 3600
+Connection ~ 12100 3600
+Wire Wire Line
+	12100 3600 12100 3700
+Wire Wire Line
+	12600 3200 12600 3100
 Wire Bus Line
 	4800 10500 11100 10500
@@
 Wire Bus Line
 	8000 5250 8000 9150
-Connection ~ 14200 3250
+Connection ~ 12600 3100
+Text Notes 11800 2650 0    50   ~ 0
+Power Supervisor\nMMP-3A package
 $EndSCHEMATC

Commit message: XIN added, PPU2 mostly done, S-SMP and S-DSP started
Parts:
- added C1: 47pF, symbol Device:C_Small
- added C2: 15pF, symbol Device:C_Small
- added C3: 10pF, symbol Device:C_Small
- added C4: 100pF, symbol Device:C_Small
- added C5: 0.01uF, symbol Device:C_Small
- added C55: (0), symbol Device:C_Small
- added C68: 56pF, symbol Device:C_Small
- added C82, C97: 0.1uF, symbol Device:C_Small
- added Q1: 2SC4699, Package_TO_SOT_SMD:SOT-323_SC-70, symbol Transistor_BJT:2SC4213
- added R1: 56K, symbol Device:R_Small
- added R2, R4: 210, symbol Device:R_Small
- added R3: 1.2K, symbol Device:R_Small
- added R5: 39, symbol Device:R_Small
- added R6: 100K, symbol Device:R_Small
- added R74: 1K, symbol Device:R_Small
- added R97: 10K, symbol Device:R_Small
- added R98: 100, symbol Device:R_Small
- added TC1: 20pF, symbol Device:CTRIM_Small
- added X1: 21.47727 MHz, Crystal:Crystal_HC49-4H_Vertical, symbol Device:Crystal_Small
- U11: footprint (none) -> SNES:MMP-3A
Connections:
- net labels added: 3.58M, HBLANK, SYSCK, VBLANK, XIN, ~IRQ, ~RESOUT0, ~RESOUT1
- net labels removed: IRQ
- wire segments 777 -> 944
- no-connect marks 50 -> 69
Other:
- moved on the sheet: P1, U13, U14, U6, U8

Commit message: Mostly complete, no ERC errors/warnings
Parts:
- added C100, C101, C102, C98, C99: 0.1uF, symbol Device:C_Small
- added C71, C72: 3pF, symbol Device:C_Small
- added C73: 47uF (10V), symbol Device:CP_Small
- added J5: Audio Out Port, symbol Connector_Generic:Conn_02x04_Counter_Clockwise
- added P4: Multi AV Out Port, symbol Connector_Generic:Conn_02x04_Counter_Clockwise
- added unit 7 of U9
- added X2: 24.576MHz, symbol Device:Crystal_Small
Connections:
- net labels added: AUDIO_LOUT, AUDIO_ROUT, CART_SOUND-L, CART_SOUND-R, MA0, MA1, MA10, MA11, MA12, MA13, MA14, MA2, MA3, MA4, MA5, MA6, MA7, MA8, MA9, MD0, MD1, MD2, MD3, MD4, MD5, MD6, MD7, REFRESH, VIDEO_B, VIDEO_G, VIDEO_R, ~CE0, ~CE1, ~MUTE, ~OE, ~VIDEO_BURST, ~VIDEO_CSYNC, ~WE
- net labels removed: 4016.D2
- wire segments 944 -> 1153
- no-connect marks 69 -> 84
Other:
- note added: "TODO: Refactor to fit this revision\nDesign S-ENC replacement"
- note added: "TODO: Reflect actual\nport to connect out to"
- note added: "TODO: connector"
- moved on the sheet: U13, U14, U15, U16

Commit message: SuperCIC added, D4 patch added
Parts:
- added LED1: GREEN, symbol Device:LED_Small
- added LED2: RED, symbol Device:LED_Small
- added RS1, RS2: 180, symbol Device:R_Small
- added RS3: 10K, symbol Device:R_Small
- added U8S: SuperCIC, Package_SO:SOIC-14_3.9x8.7mm_P1.27mm, symbol SNES:SuperCIC
- added UP1: 74LS125, symbol 74xx:74LS04
- added UP2: 74LS133, symbol 74xx:74LS133
- added UP3: 74LS125, symbol 74xx:74LS125
- P4: value Multi AV Out Port -> Multi AV Out
- U9: footprint (none) -> Package_SO:SOIC-14_3.9x8.7mm_P1.27mm
Connections:
- net labels added: $214F_PATCH, CIC_CL1, CIC_RESET
- wire segments 1153 -> 1242
Other:
- note added: "CIC no stuff / SuperCIC"
- note added: "Connect to S-ENC sub-board"
- note added: "Connect to amplifier sub-board"
- note added: "DC Power Input\nUSB +5V @ 1.7A, derived from +10V @ 0.85A"
- note added: "SuperCIC $213f patching (D4 pin)"
- note removed: "DC Power Input\nUSB +5V @ 1.7A\nDerived from +10V @ 0.85A"
- note removed: "TODO: Refactor to fit this revision\nDesign S-ENC replacement"
- note removed: "TODO: Reflect actual\nport to connect out to"

Commit message: Capacitor footprints added
Parts:
- C1, C100, C101, C102, C107, C2, C29, C3, C31, C35, C36, C37, C38, C39, C4, C40, C41, C42, C43, C5, C55, C68, C70, C71, C72, C82, C89, C90, C91, C92, C93, C94, C95, C97, C98, C99: footprint (none) -> Capacitor_SMD:C_0603_1608Metric
Changed lines of the file:
@@
 F 0 "C38" V 5000 2200 50  0000 L CNN
 F 1 "330pF" V 5500 2500 50  0000 C CNN
-F 2 "" H 5000 2800 50  0001 C CNN
+F 2 "Capacitor_SMD:C_0603_1608Metric" H 5000 2800 50  0001 C CNN
 F 3 "~" H 5000 2800 50  0001 C CNN
 	1    5000 2800
@@
 F 0 "C43" V 6900 2200 50  0000 L CNN
 F 1 "330pF" V 7400 2500 50  0000 C CNN
-F 2 "" H 6900 2800 50  0001 C CNN
+F 2 "Capacitor_SMD:C_0603_1608Metric" H 6900 2800 50  0001 C CNN
 F 3 "~" H 6900 2800 50  0001 C CNN
 	1    6900 2800
@@
 F 0 "C107" V 5200 1800 50  0000 C CNN
 F 1 "0.01uF" V 5000 1800 50  0000 C CNN
-F 2 "" H 5100 1800 50  0001 C CNN
+F 2 "Capacitor_SMD:C_0603_1608Metric" H 5100 1800 50  0001 C CNN
 F 3 "~" H 5100 1800 50  0001 C CNN
 	1    5100 1800
@@
 F 0 "C35" V 6500 2200 50  0000 L CNN
 F 1 "330pF" V 7000 2500 50  0000 C CNN
-F 2 "" H 6500 2800 50  0001 C CNN
+F 2 "Capacitor_SMD:C_0603_1608Metric" H 6500 2800 50  0001 C CNN
 F 3 "~" H 6500 2800 50  0001 C CNN
 	1    6500 2800
@@
 F 0 "C90" V 4350 5650 50  0000 C CNN
 F 1 "0.1uF" V 4050 5650 50  0000 C CNN
-F 2 "" H 4200 5650 50  0001 C CNN
+F 2 "Capacitor_SMD:C_0603_1608Metric" H 4200 5650 50  0001 C CNN
 F 3 "~" H 4200 5650 50  0001 C CNN
 	1    4200 5650
@@
 F 0 "C91" V 7750 5650 50  0000 C CNN
 F 1 "0.1uF" V 7450 5650 50  0000 C CNN
-F 2 "" H 7600 5650 50  0001 C CNN
+F 2 "Capacitor_SMD:C_0603_1608Metric" H 7600 5650 50  0001 C CNN
 F 3 "~" H 7600 5650 50  0001 C CNN
 	1    7600 5650
@@
 F 0 "C93" V 8850 5450 50  0000 C CNN
 F 1 "0.1uF" V 8850 5700 50  0000 C CNN
-F 2 "" H 8750 5550 50  0001 C CNN
+F 2 "Capacitor_SMD:C_0603_1608Metric" H 8750 5550 50  0001 C CNN
 F 3 "~" H 8750 5550 50  0001 C CNN
 	1    8750 5550
@@
 F 0 "C94" V 8850 7950 50  0000 C CNN
 F 1 "0.1uF" V 8850 8200 50  0000 C CNN
-F 2 "" H 8750 8050 50  0001 C CNN
+F 2 "Capacitor_SMD:C_0603_1608Metric" H 8750 8050 50  0001 C CNN
 F 3 "~" H 8750 8050 50  0001 C CNN
 	1    8750 8050
@@
 F 0 "C37" V 6600 2600 50  0000 L CNN
 F 1 "330pF" V 7100 2800 50  0000 C CNN
-F 2 "" H 6600 3000 50  0001 C CNN
+F 2 "Capacitor_SMD:C_0603_1608Metric" H 6600 3000 50  0001 C CNN
 F 3 "~" H 6600 3000 50  0001 C CNN
 	1    6600 3000
@@
 F 0 "C39" V 6700 2200 50  0000 L CNN
 F 1 "330pF" V 7200 2500 50  0000 C CNN
-F 2 "" H 6700 2800 50  0001 C CNN
+F 2 "Capacitor_SMD:C_0603_1608Metric" H 6700 2800 50  0001 C CNN
 F 3 "~" H 6700 2800 50  0001 C CNN
 	1    6700 2800
@@
 F 0 "C41" V 6800 2600 50  0000 L CNN
 F 1 "330pF" V 7300 2800 50  0000 C CNN
-F 2 "" H 6800 3000 50  0001 C CNN
+F 2 "Capacitor_SMD:C_0603_1608Metric" H 6800 3000 50  0001 C CNN
 F 3 "~" H 6800 3000 50  0001 C CNN
 	1    6800 3000
@@
 F 0 "C40" V 5100 3400 50  0000 R CNN
 F 1 "330pF" V 5600 3200 50  0000 C CNN
-F 2 "" H 5100 3000 50  0001 C CNN
+F 2 "Capacitor_SMD:C_0603_1608Metric" H 5100 3000 50  0001 C CNN
 F 3 "~" H 5100 3000 50  0001 C CNN
 	1    5100 3000
@@
 F 0 "C42" V 5200 2200 50  0000 L CNN
 F 1 "330pF" V 5700 2500 50  0000 C CNN
-F 2 "" H 5200 2800 50  0001 C CNN
+F 2 "Capacitor_SMD:C_0603_1608Metric" H 5200 2800 50  0001 C CNN
 F 3 "~" H 5200 2800 50  0001 C CNN
 	1    5200 2800
@@
 F 0 "C36" V 4900 2600 50  0000 L CNN
 F 1 "330pF" V 5400 2800 50  0000 C CNN
-F 2 "" H 4900 3000 50  0001 C CNN
+F 2 "Capacitor_SMD:C_0603_1608Metric" H 4900 3000 50  0001 C CNN
 F 3 "~" H 4900 3000 50  0001 C CNN
 	1    4900 3000
@@
 F 0 "C95" V 4100 12500 50  0000 C TNN
 F 1 "0.1uF" V 3900 12500 50  0000 C BNN
-F 2 "" H 4000 12500 50  0001 C CNN
+F 2 "Capacitor_SMD:C_0603_1608Metric" H 4000 12500 50  0001 C CNN
 F 3 "~" H 4000 12500 50  0001 C CNN
 	1    4000 12500
@@
 F 0 "C92" V 13450 5650 50  0000 C CNN
 F 1 "0.1uF" V 13150 5650 50  0000 C CNN
-F 2 "" H 13300 5650 50  0001 C CNN
+F 2 "Capacitor_SMD:C_0603_1608Metric" H 13300 5650 50  0001 C CNN
 F 3 "~" H 13300 5650 50  0001 C CNN
 	1    13300 5650
@@
 F 0 "C29" H 2092 18046 50  0000 L CNN
 F 1 "0.1uF" H 2092 17955 50  0000 L CNN
-F 2 "" H 2000 18000 50  0001 C CNN
+F 2 "Capacitor_SMD:C_0603_1608Metric" H 2000 18000 50  0001 C CNN
 F 3 "~" H 2000 18000 50  0001 C CNN
 	1    2000 18000
@@
 F 0 "C70" H 5692 17696 50  0000 L CNN
 F 1 "82pF" H 5692 17605 50  0000 L CNN
-F 2 "" H 5600 17650 50  0001 C CNN
+F 2 "Capacitor_SMD:C_0603_1608Metric" H 5600 17650 50  0001 C CNN
 F 3 "~" H 5600 17650 50  0001 C CNN
 	1    5600 17650
@@
 F 0 "C89" H 11792 2246 50  0000 L CNN
 F 1 "100nF" H 11792 2155 50  0000 L CNN
-F 2 "" H 11700 2200 50  0001 C CNN
+F 2 "Capacitor_SMD:C_0603_1608Metric" H 11700 2200 50  0001 C CNN
 F 3 "~" H 11700 2200 50  0001 C CNN
 	1    11700 2200
@@
 F 0 "C2" V 15500 2850 50  0000 L CNN
 F 1 "15pF" V 15700 3000 50  0000 C CNN
-F 2 "" H 15600 3000 50  0001 C CNN
+F 2 "Capacitor_SMD:C_0603_1608Metric" H 15600 3000 50  0001 C CNN
 F 3 "~" H 15600 3000 50  0001 C CNN
 	1    15600 3000
@@
 F 0 "C5" H 15092 3946 50  0000 L CNN
 F 1 "0.01uF" H 15092 3855 50  0000 L CNN
-F 2 "" H 15000 3900 50  0001 C CNN
+F 2 "Capacitor_SMD:C_0603_1608Metric" H 15000 3900 50  0001 C CNN
 F 3 "~" H 15000 3900 50  0001 C CNN
 	1    15000 3900
@@
 F 0 "C3" H 14592 3946 50  0000 L CNN
 F 1 "10pF" H 14592 3855 50  0000 L CNN
-F 2 "" H 14500 3900 50  0001 C CNN
+F 2 "Capacitor_SMD:C_0603_1608Metric" H 14500 3900 50  0001 C CNN
 F 3 "~" H 14500 3900 50  0001 C CNN
 	1    14500 3900
@@
 F 0 "C4" V 14450 3100 50  0000 C CNN
 F 1 "100pF" V 14150 3100 50  0000 C CNN
-F 2 "" H 14300 3100 50  0001 C CNN
+F 2 "Capacitor_SMD:C_0603_1608Metric" H 14300 3100 50  0001 C CNN
 F 3 "~" H 14300 3100 50  0001 C CNN
 	1    14300 3100
@@
 F 0 "C82" H 14792 2746 50  0000 L CNN
 F 1 "0.1uF" H 14792 2655 50  0000 L CNN
-F 2 "" H 14700 2700 50  0001 C CNN
+F 2 "Capacitor_SMD:C_0603_1608Metric" H 14700 2700 50  0001 C CNN
 F 3 "~" H 14700 2700 50  0001 C CNN
 	1    14700 2700
@@
 F 0 "C1" H 15892 3946 50  0000 L CNN
 F 1 "47pF" H 15892 3855 50  0000 L CNN
-F 2 "" H 15800 3900 50  0001 C CNN
+F 2 "Capacitor_SMD:C_0603_1608Metric" H 15800 3900 50  0001 C CNN
 F 3 "~" H 15800 3900 50  0001 C CNN
 	1    15800 3900
@@
 F 0 "C68" V 10950 8200 50  0000 L BNN
 F 1 "56pF" V 10800 8150 50  0000 L TNN
-F 2 "" H 11000 8150 50  0001 C CNN
+F 2 "Capacitor_SMD:C_0603_1608Metric" H 11000 8150 50  0001 C CNN
 F 3 "~" H 11000 8150 50  0001 C CNN
 	1    11000 8150
@@
 F 0 "C97" H 11892 14796 50  0000 L CNN
 F 1 "0.1uF" H 11892 14705 50  0000 L CNN
-F 2 "" H 11800 14750 50  0001 C CNN
+F 2 "Capacitor_SMD:C_0603_1608Metric" H 11800 14750 50  0001 C CNN
 F 3 "~" H 11800 14750 50  0001 C CNN
 	1    11800 14750
@@
 F 0 "C55" H 9950 14350 50  0000 R CNN
 F 1 "(0)" H 10150 14350 50  0000 R CNN
-F 2 "" H 10000 14250 50  0001 C CNN
+F 2 "Capacitor_SMD:C_0603_1608Metric" H 10000 14250 50  0001 C CNN
 F 3 "~" H 10000 14250 50  0001 C CNN
 	1    10000 14250
@@
 F 0 "C101" V 15100 13800 50  0000 R CNN
 F 1 "0.1uF" V 15100 14100 50  0000 R CNN
-F 2 "" H 15200 13850 50  0001 C CNN
+F 2 "Capacitor_SMD:C_0603_1608Metric" H 15200 13850 50  0001 C CNN
 F 3 "~" H 15200 13850 50  0001 C CNN
 	1    15200 13850
@@
 F 0 "C100" V 15100 16100 50  0000 R CNN
 F 1 "0.1uF" V 15100 16400 50  0000 R CNN
-F 2 "" H 15200 16150 50  0001 C CNN
+F 2 "Capacitor_SMD:C_0603_1608Metric" H 15200 16150 50  0001 C CNN
 F 3 "~" H 15200 16150 50  0001 C CNN
 	1    15200 16150
@@
 F 0 "C99" V 13400 13550 50  0000 C CNN
 F 1 "0.1uF" V 13600 13550 50  0000 C CNN
-F 2 "" H 13500 13550 50  0001 C CNN
+F 2 "Capacitor_SMD:C_0603_1608Metric" H 13500 13550 50  0001 C CNN
 F 3 "~" H 13500 13550 50  0001 C CNN
 	1    13500 13550
@@
 F 0 "C31" H 18150 5500 50  0000 L CNN
 F 1 "0.01uF 50V" H 18350 5600 50  0000 C CNN
-F 2 "" H 18400 5500 50  0001 C CNN
+F 2 "Capacitor_SMD:C_0603_1608Metric" H 18400 5500 50  0001 C CNN
 F 3 "~" H 18400 5500 50  0001 C CNN
 	1    18400 5500
@@
 F 0 "C98" V 13000 13550 50  0000 C CNN
 F 1 "0.1uF" V 13200 13550 50  0000 C CNN
-F 2 "" H 13100 13550 50  0001 C CNN
+F 2 "Capacitor_SMD:C_0603_1608Metric" H 13100 13550 50  0001 C CNN
 F 3 "~" H 13100 13550 50  0001 C CNN
 	1    13100 13550
@@
 F 0 "C71" H 11600 13450 50  0000 C TNN
 F 1 "3pF" H 11600 13600 50  0000 C TNN
-F 2 "" H 11700 13500 50  0001 C CNN
+F 2 "Capacitor_SMD:C_0603_1608Metric" H 11700 13500 50  0001 C CNN
 F 3 "~" H 11700 13500 50  0001 C CNN
 	1    11700 13500
@@
 F 0 "C72" H 11200 13450 50  0000 C TNN
 F 1 "3pF" H 11000 13600 50  0000 C TNN
-F 2 "" H 11100 13500 50  0001 C CNN
+F 2 "Capacitor_SMD:C_0603_1608Metric" H 11100 13500 50  0001 C CNN
 F 3 "~" H 11100 13500 50  0001 C CNN
 	1    11100 13500
@@
 F 0 "C102" V 15271 11950 50  0000 C CNN
 F 1 "0.1uF" V 15362 11950 50  0000 C CNN
-F 2 "" H 15500 11950 50  0001 C CNN
+F 2 "Capacitor_SMD:C_0603_1608Metric" H 15500 11950 50  0001 C CNN
 F 3 "~" H 15500 11950 50  0001 C CNN
 	1    15500 11950
@@
 Wire Bus Line
 	14400 14250 14400 17950
+Entry Bus Bus
+	9850 4600 9950 4700
 $EndSCHEMATC

Commit message: Most footprints added
Parts:
- added unit 7 of UP1
- added unit 2 of UP2
- added unit 5 of UP3
- C67: footprint (none) -> Capacitor_SMD:CP_Elec_10x12.6
- C73: footprint (none) -> Capacitor_SMD:CP_Elec_6.3x5.4
- J5, P4: footprint (none) -> Connector_PinHeader_1.27mm:PinHeader_2x04_P1.27mm_Vertical
- LED1, LED2: footprint (none) -> LED_SMD:LED_1206_3216Metric
- RN7781, RN7882, RN8490: footprint Resistor_SMD:R_Array_Convex_4x0603 -> Resistor_SMD:R_Array_Convex_4x1206
- RN8391: footprint (none) -> Resistor_SMD:R_Array_Convex_5x1206
- TC1: footprint (none) -> Capacitor_SMD:C_Trimmer_Murata_TZB4-A
- UP1, UP3: footprint (none) -> Package_SO:SOIC-14_3.9x8.7mm_P1.27mm
- UP2: footprint (none) -> Package_SO:SOIC-16_3.9x9.9mm_P1.27mm
- renumbered U8S to US8
Connections:
- wire segments 1242 -> 1254

Commit message: Resistor footprints added
Parts:
- R1, R2, R3, R4, R5, R6, R74, R75, R97, R98: footprint (none) -> Resistor_SMD:R_0603_1608Metric
Changed lines of the file:
@@
 F 0 "R75" H 10642 1754 50  0000 R CNN
 F 1 "100K" H 10642 1845 50  0000 R CNN
-F 2 "" H 10700 1800 50  0001 C CNN
+F 2 "Resistor_SMD:R_0603_1608Metric" H 10700 1800 50  0001 C CNN
 F 3 "~" H 10700 1800 50  0001 C CNN
 	1    10700 1800
@@
 F 0 "R1" H 15342 3154 50  0000 R CNN
 F 1 "56K" H 15342 3245 50  0000 R CNN
-F 2 "" H 15400 3200 50  0001 C CNN
+F 2 "Resistor_SMD:R_0603_1608Metric" H 15400 3200 50  0001 C CNN
 F 3 "~" H 15400 3200 50  0001 C CNN
 	1    15400 3200
@@
 F 0 "R2" H 15342 3854 50  0000 R CNN
 F 1 "210" H 15342 3945 50  0000 R CNN
-F 2 "" H 15400 3900 50  0001 C CNN
+F 2 "Resistor_SMD:R_0603_1608Metric" H 15400 3900 50  0001 C CNN
 F 3 "~" H 15400 3900 50  0001 C CNN
 	1    15400 3900
@@
 F 0 "R5" V 12500 3100 50  0000 C CNN
 F 1 "39" V 12300 3100 50  0000 C CNN
-F 2 "" H 12400 3100 50  0001 C CNN
+F 2 "Resistor_SMD:R_0603_1608Metric" H 12400 3100 50  0001 C CNN
 F 3 "~" H 12400 3100 50  0001 C CNN
 	1    12400 3100
@@
 F 0 "R4" H 12142 3254 50  0000 R CNN
 F 1 "210" H 12142 3345 50  0000 R CNN
-F 2 "" H 12200 3300 50  0001 C CNN
+F 2 "Resistor_SMD:R_0603_1608Metric" H 12200 3300 50  0001 C CNN
 F 3 "~" H 12200 3300 50  0001 C CNN
 	1    12200 3300
@@
 F 0 "R6" V 13600 2850 50  0000 L CNN
 F 1 "100K" V 13600 2800 50  0000 R CNN
-F 2 "" H 13700 2800 50  0001 C CNN
+F 2 "Resistor_SMD:R_0603_1608Metric" H 13700 2800 50  0001 C CNN
 F 3 "~" H 13700 2800 50  0001 C CNN
 	1    13700 2800
@@
 F 0 "R3" H 14942 2654 50  0000 R CNN
 F 1 "1.2K" H 14942 2745 50  0000 R CNN
-F 2 "" H 15000 2700 50  0001 C CNN
+F 2 "Resistor_SMD:R_0603_1608Metric" H 15000 2700 50  0001 C CNN
 F 3 "~" H 15000 2700 50  0001 C CNN
 	1    15000 2700
@@
 F 0 "R74" H 10759 5446 50  0000 L CNN
 F 1 "1K" H 10759 5355 50  0000 L CNN
-F 2 "" H 10700 5400 50  0001 C CNN
+F 2 "Resistor_SMD:R_0603_1608Metric" H 10700 5400 50  0001 C CNN
 F 3 "~" H 10700 5400 50  0001 C CNN
 	1    10700 5400
@@
 F 0 "R97" H 6150 12650 50  0000 R CNN
 F 1 "10K" H 6150 12550 50  0000 R CNN
-F 2 "" H 6200 12600 50  0001 C CNN
+F 2 "Resistor_SMD:R_0603_1608Metric" H 6200 12600 50  0001 C CNN
 F 3 "~" H 6200 12600 50  0001 C CNN
 	1    6200 12600
@@
 F 0 "R98" V 10950 7600 50  0000 R BNN
 F 1 "100" V 10950 7750 50  0000 C BNN
-F 2 "" H 11000 7650 50  0001 C CNN
+F 2 "Resistor_SMD:R_0603_1608Metric" H 11000 7650 50  0001 C CNN
 F 3 "~" H 11000 7650 50  0001 C CNN
 	1    11000 7650
