File: MainBoard.sch (KiCad schematic (older format))
At the start: 100 parts, among them J1 USB B Mini, J5 Audio Out Port, P1 CARTRIDGE_SLOT, P2 FRONT_PANEL_CONNECTOR, P4 Multi AV Out, Q1 2SC4699, SW1 RESET, U1 S-CPU, U11 PST529D, U13 S-SMP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

Commit message: Missing footprints added
Parts:
- C62: footprint (none) -> Capacitor_SMD:CP_Elec_6.3x5.4
- J1: footprint (none) -> Connector_USB:USB_Mini-B_Lumberg_2486_01_Horizontal
- RS1, RS2, RS3: footprint (none) -> Resistor_SMD:R_0603_1608Metric
- U13: footprint (none) -> SNES:PQFP-64_14x20mm_P1.0mm
- X2: footprint (none) -> Crystal:Crystal_SMD_HC49-SD
Changed lines of the file:
@@
 F 0 "U13" H 10800 14650 50  0000 L CNN
 F 1 "S-SMP" H 11100 11350 50  0000 C CNN
-F 2 "" H 11100 14650 50  0001 C CNN
+F 2 "SNES:PQFP-64_14x20mm_P1.0mm" H 11100 14650 50  0001 C CNN
 F 3 "" H 11100 14650 50  0001 C CNN
 	1    11100 14650
@@
 F 0 "C62" H 2350 17600 50  0000 L CNN
 F 1 "2.2uF" H 2350 17400 50  0000 L CNN
-F 2 "" H 2300 17500 50  0001 C CNN
+F 2 "Capacitor_SMD:CP_Elec_6.3x5.4" H 2300 17500 50  0001 C CNN
 F 3 "~" H 2300 17500 50  0001 C CNN
 	1    2300 17500
@@
 F 0 "J1" H 19400 5750 50  0000 C CNN
 F 1 "USB B Mini" H 19400 5650 50  0000 C CNN
-F 2 "" H 19550 5250 50  0001 C CNN
+F 2 "Connector_USB:USB_Mini-B_Lumberg_2486_01_Horizontal" H 19550 5250 50  0001 C CNN
 F 3 "~" H 19550 5250 50  0001 C CNN
 	1    19400 5300
@@
 F 0 "X2" H 11400 13500 50  0000 C BNN
 F 1 "24.576MHz" H 11400 13400 50  0000 C BNN
-F 2 "" H 11400 13300 50  0001 C CNN
+F 2 "Crystal:Crystal_SMD_HC49-SD" H 11400 13300 50  0001 C CNN
 F 3 "~" H 11400 13300 50  0001 C CNN
 	1    11400 13300
@@
 F 0 "RS1" V 2550 19950 50  0000 C BNN
 F 1 "180" V 2550 20150 50  0000 C BNN
-F 2 "" H 2600 20050 50  0001 C CNN
+F 2 "Resistor_SMD:R_0603_1608Metric" H 2600 20050 50  0001 C CNN
 F 3 "~" H 2600 20050 50  0001 C CNN
 	1    2600 20050
@@
 F 0 "RS2" V 2500 20050 50  0000 C TNN
 F 1 "180" V 2500 19850 50  0000 C TNN
-F 2 "" H 2600 19950 50  0001 C CNN
+F 2 "Resistor_SMD:R_0603_1608Metric" H 2600 19950 50  0001 C CNN
 F 3 "~" H 2600 19950 50  0001 C CNN
 	1    2600 19950
@@
 F 0 "RS3" V 4100 20350 50  0000 C CNN
 F 1 "10K" V 4100 20150 50  0000 C CNN
-F 2 "" H 4200 20250 50  0001 C CNN
+F 2 "Resistor_SMD:R_0603_1608Metric" H 4200 20250 50  0001 C CNN
 F 3 "~" H 4200 20250 50  0001 C CNN
 	1    4200 20250
@@
 $EndComp
 $Comp
-L power:VCC #PWR?
+L power:VCC #PWR0197
 U 1 1 611D47D6
 P 6500 21400
-F 0 "#PWR?" H 6500 21250 50  0001 C CNN
+F 0 "#PWR0197" H 6500 21250 50  0001 C CNN
 F 1 "VCC" H 6515 21573 50  0000 C CNN
 F 2 "" H 6500 21400 50  0001 C CNN
@@
 	6500 21500 6600 21500
 $Comp
-L power:VCC #PWR?
+L power:VCC #PWR0198
 U 1 1 613ADA19
 P 7800 21400
-F 0 "#PWR?" H 7800 21250 50  0001 C CNN
+F 0 "#PWR0198" H 7800 21250 50  0001 C CNN
 F 1 "VCC" H 7815 21573 50  0000 C CNN
 F 2 "" H 7800 21400 50  0001 C CNN
@@
 	7800 21500 7900 21500
 $Comp
-L power:GND #PWR?
+L power:GND #PWR0199
 U 1 1 6158882B
 P 7700 21600
-F 0 "#PWR?" H 7700 21350 50  0001 C CNN
+F 0 "#PWR0199" H 7700 21350 50  0001 C CNN
 F 1 "GND" H 7705 21427 50  0000 C CNN
 F 2 "" H 7700 21600 50  0001 C CNN
@@
 	7700 21500 7600 21500
 $Comp
-L power:GND #PWR?
+L power:GND #PWR0200
 U 1 1 61B1A80D
 P 9000 21600
-F 0 "#PWR?" H 9000 21350 50  0001 C CNN
+F 0 "#PWR0200" H 9000 21350 50  0001 C CNN
 F 1 "GND" H 9005 21427 50  0000 C CNN
 F 2 "" H 9000 21600 50  0001 C CNN
@@
 	9000 21500 8900 21500
 $Comp
-L power:VCC #PWR?
+L power:VCC #PWR0201
 U 1 1 61CF7C21
 P 9100 21400
-F 0 "#PWR?" H 9100 21250 50  0001 C CNN
+F 0 "#PWR0201" H 9100 21250 50  0001 C CNN
 F 1 "VCC" H 9115 21573 50  0000 C CNN
 F 2 "" H 9100 21400 50  0001 C CNN
@@
 	9100 21500 9200 21500
 $Comp
-L power:GND #PWR?
+L power:GND #PWR0202
 U 1 1 61ED654C
 P 10300 21600
-F 0 "#PWR?" H 10300 21350 50  0001 C CNN
+F 0 "#PWR0202" H 10300 21350 50  0001 C CNN
 F 1 "GND" H 10305 21427 50  0000 C CNN
 F 2 "" H 10300 21600 50  0001 C CNN

Commit message: Notes errata, 213f PLD version added
Parts:
- added CPA1: 100nF, symbol Device:C_Small
- added UPA1: 16V8, Package_LCC:PLCC-20, symbol Logic_Programmable:GAL16V8
Connections:
- wire segments 1254 -> 1279
- no-connect marks 84 -> 88
Other:
- note added: "CIC no stuff / SuperCIC\nby ikari_01"
- note added: "SuperCIC $213f patch PLD alt\nby FFVIMan & Niluje\n\nJED source and binary can be found in repository"
- note added: "SuperCIC $213f patching (D4 pin)\nby ikari_01 (2012)"
- note added: "TODO:\nresearch for circuit replacement"
- note added: "TODO:\nresearch for replacement"
- note removed: "CIC no stuff / SuperCIC"
- note removed: "SuperCIC $213f patching (D4 pin)"
- note removed: "TODO: connector"

Commit message: Missing footprint added, Notes errata
Parts:
- CPA1: footprint (none) -> Capacitor_SMD:C_0603_1608Metric
Other:
- note added: "Roughly 2.3~~2.4V\nsquare signal output"
Changed lines of the file:
@@
 $EndComp
 $Comp
-L power:VCC #PWR?
+L power:VCC #PWR0203
 U 1 1 606C34F9
 P 13400 19650
-F 0 "#PWR?" H 13400 19500 50  0001 C CNN
+F 0 "#PWR0203" H 13400 19500 50  0001 C CNN
 F 1 "VCC" H 13500 19650 50  0000 C CNN
 F 2 "" H 13400 19650 50  0001 C CNN
@@
 	13400 19650 13400 19750
 $Comp
-L power:GND #PWR?
+L power:GND #PWR0204
 U 1 1 608A5989
 P 13400 21350
-F 0 "#PWR?" H 13400 21100 50  0001 C CNN
+F 0 "#PWR0204" H 13400 21100 50  0001 C CNN
 F 1 "GND" H 13405 21177 50  0000 C CNN
 F 2 "" H 13400 21350 50  0001 C CNN
@@
 F 0 "CPA1" V 13800 21250 50  0000 C CNN
 F 1 "100nF" V 13550 21250 50  0000 C TNN
-F 2 "" H 13700 21250 50  0001 C CNN
+F 2 "Capacitor_SMD:C_0603_1608Metric" H 13700 21250 50  0001 C CNN
 F 3 "~" H 13700 21250 50  0001 C CNN
 	1    13700 21250
@@
 	13400 21250 13400 21150
 $Comp
-L power:VCC #PWR?
+L power:VCC #PWR0205
 U 1 1 6102D62E
 P 13900 21150
-F 0 "#PWR?" H 13900 21000 50  0001 C CNN
+F 0 "#PWR0205" H 13900 21000 50  0001 C CNN
 F 1 "VCC" H 13915 21323 50  0000 C CNN
 F 2 "" H 13900 21150 50  0001 C CNN
@@
 Wire Wire Line
 	11800 3500 11800 5000
-Wire Bus Line
-	5000 11400 11300 11400
-Wire Bus Line
-	4800 11600 11100 11600
-Wire Bus Line
-	4600 12000 8100 12000
-Wire Bus Line
-	4400 12200 7900 12200
-Wire Bus Line
-	11200 8950 11200 11500
-Wire Wire Line
-	7500 14800 8700 14800
-Wire Wire Line
-	3900 9850 5200 9850
-Wire Bus Line
-	5000 16200 7900 16200
-Wire Wire Line
-	3700 14400 4800 14400
-Wire Wire Line
-	3900 9050 4800 9050
-Wire Wire Line
-	3900 8850 4600 8850
-Wire Bus Line
-	5800 5300 5800 8650
-Wire Bus Line
-	5900 15500 5900 16100
-Wire Bus Line
-	2200 12100 2200 15400
-Wire Bus Line
-	8200 12100 8200 14800
-Wire Bus Line
-	8000 15500 8000 16100
-Wire Bus Line
-	9400 11700 9400 17250
-Wire Bus Line
-	9100 11500 9100 17650
-Wire Bus Line
-	14200 13650 14200 14650
-Wire Bus Line
-	4500 6150 4500 11900
-Wire Bus Line
-	8800 11300 8800 14700
-Wire Bus Line
-	9800 5300 9800 8550
-Wire Bus Line
-	9500 2300 9500 3900
-Wire Bus Line
-	1500 2400 1500 4000
-Wire Bus Line
-	4700 8950 4700 14500
-Wire Bus Line
-	16200 13650 16200 16850
-Wire Bus Line
-	14100 16650 14100 18150
-Wire Bus Line
-	10000 14900 10000 17050
-Wire Bus Line
-	11400 9150 11400 11300
-Wire Bus Line
-	11600 9950 11600 11100
-Wire Bus Line
-	1600 4100 1600 8250
-Wire Bus Line
-	5600 5200 5600 7450
-Wire Bus Line
-	8000 12300 8000 14200
-Wire Bus Line
-	11500 5200 11500 7450
-Wire Bus Line
-	5800 12300 5800 14200
-Wire Bus Line
-	16000 14950 16000 18150
-Wire Bus Line
-	5300 9950 5300 15400
-Wire Bus Line
-	4900 9150 4900 16100
-Wire Bus Line
-	2400 12300 2400 14600
-Wire Bus Line
-	9600 6650 9600 10750
-Wire Bus Line
-	7700 9150 7700 10750
-Wire Bus Line
-	4300 6550 4300 12100
-Wire Bus Line
-	13500 8350 13500 11700
-Wire Bus Line
-	8000 5950 8000 9850
-Wire Bus Line
-	14400 14250 14400 17950
 Text Notes 16000 2500 2    50   ~ 0
 TODO:\nresearch for circuit replacement
+Wire Bus Line
+	5000 11400 11300 11400
+Wire Bus Line
+	4800 11600 11100 11600
+Wire Bus Line
+	4600 12000 8100 12000
+Wire Bus Line
+	4400 12200 7900 12200
+Wire Bus Line
+	11200 8950 11200 11500
+Wire Wire Line
+	7500 14800 8700 14800
+Wire Wire Line
+	3900 9850 5200 9850
+Wire Bus Line
+	5000 16200 7900 16200
+Wire Wire Line
+	3700 14400 4800 14400
+Wire Wire Line
+	3900 9050 4800 9050
+Wire Wire Line
+	3900 8850 4600 8850
+Wire Bus Line
+	5800 5300 5800 8650
+Wire Bus Line
+	5900 15500 5900 16100
+Wire Bus Line
+	2200 12100 2200 15400
+Wire Bus Line
+	8200 12100 8200 14800
+Wire Bus Line
+	8000 15500 8000 16100
+Wire Bus Line
+	9400 11700 9400 17250
+Wire Bus Line
+	9100 11500 9100 17650
+Wire Bus Line
+	14200 13650 14200 14650
+Wire Bus Line
+	4500 6150 4500 11900
+Wire Bus Line
+	8800 11300 8800 14700
+Wire Bus Line
+	9800 5300 9800 8550
+Wire Bus Line
+	9500 2300 9500 3900
+Wire Bus Line
+	1500 2400 1500 4000
+Wire Bus Line
+	4700 8950 4700 14500
+Wire Bus Line
+	16200 13650 16200 16850
+Wire Bus Line
+	14100 16650 14100 18150
+Wire Bus Line
+	10000 14900 10000 17050
+Wire Bus Line
+	11400 9150 11400 11300
+Wire Bus Line
+	11600 9950 11600 11100
+Wire Bus Line
+	1600 4100 1600 8250
+Wire Bus Line
+	5600 5200 5600 7450
+Wire Bus Line
+	8000 12300 8000 14200
+Wire Bus Line
+	11500 5200 11500 7450
+Wire Bus Line
+	5800 12300 5800 14200
+Wire Bus Line
+	16000 14950 16000 18150
+Wire Bus Line
+	5300 9950 5300 15400
+Wire Bus Line
+	4900 9150 4900 16100
+Wire Bus Line
+	2400 12300 2400 14600
+Wire Bus Line
+	9600 6650 9600 10750
+Wire Bus Line
+	7700 9150 7700 10750
+Wire Bus Line
+	4300 6550 4300 12100
+Wire Bus Line
+	13500 8350 13500 11700
+Wire Bus Line
+	8000 5950 8000 9850
+Wire Bus Line
+	14400 14250 14400 17950
+Text Notes 11800 3200 0    50   ~ 0
+Roughly 2.3~~2.4V\nsquare signal output
 $EndSCHEMATC

Commit message: Fixed multiple footprints for UP3
Parts:
- F1: footprint Fuse:Fuse_1812_4532Metric -> Fuse:Fuse_1206_3216Metric
Changed lines of the file:
@@
 F 0 "F1" V 18600 5100 50  0000 C CNN
 F 1 "Polyfuse" V 18800 5100 50  0000 C CNN
-F 2 "Fuse:Fuse_1812_4532Metric" H 18750 4900 50  0001 L CNN
+F 2 "Fuse:Fuse_1206_3216Metric" H 18750 4900 50  0001 L CNN
 F 3 "~" H 18700 5100 50  0001 C CNN
 	1    18700 5100
@@
 $EndComp
 $Comp
-L 74xx:74LS125 UP3
-U 5 1 604D413B
-P 10700 21500
-F 0 "UP3" V 10450 21600 50  0000 L CNN
-F 1 "74LS125" V 10950 21450 50  0000 L CNN
-F 2 "Package_SO:SOIC-14_3.9x8.7mm_P1.27mm" H 10700 21500 50  0001 C CNN
-F 3 "http://www.ti.com/lit/gpn/sn74LS126a" H 10700 21500 50  0001 C CNN
-	5    10700 21500
-	0    -1   1    0
-$EndComp
-$Comp
 L power:VCC #PWR0197
 U 1 1 611D47D6
@@
 Text Notes 16000 2500 2    50   ~ 0
 TODO:\nresearch for circuit replacement
-Wire Bus Line
-	5000 11400 11300 11400
-Wire Bus Line
-	4800 11600 11100 11600
-Wire Bus Line
-	4600 12000 8100 12000
-Wire Bus Line
-	4400 12200 7900 12200
-Wire Bus Line
-	11200 8950 11200 11500
-Wire Wire Line
-	7500 14800 8700 14800
-Wire Wire Line
-	3900 9850 5200 9850
-Wire Bus Line
-	5000 16200 7900 16200
-Wire Wire Line
-	3700 14400 4800 14400
-Wire Wire Line
-	3900 9050 4800 9050
-Wire Wire Line
-	3900 8850 4600 8850
-Wire Bus Line
-	5800 5300 5800 8650
-Wire Bus Line
-	5900 15500 5900 16100
-Wire Bus Line
-	2200 12100 2200 15400
-Wire Bus Line
-	8200 12100 8200 14800
-Wire Bus Line
-	8000 15500 8000 16100
-Wire Bus Line
-	9400 11700 9400 17250
-Wire Bus Line
-	9100 11500 9100 17650
-Wire Bus Line
-	14200 13650 14200 14650
-Wire Bus Line
-	4500 6150 4500 11900
-Wire Bus Line
-	8800 11300 8800 14700
-Wire Bus Line
-	9800 5300 9800 8550
-Wire Bus Line
-	9500 2300 9500 3900
-Wire Bus Line
-	1500 2400 1500 4000
-Wire Bus Line
-	4700 8950 4700 14500
-Wire Bus Line
-	16200 13650 16200 16850
-Wire Bus Line
-	14100 16650 14100 18150
-Wire Bus Line
-	10000 14900 10000 17050
-Wire Bus Line
-	11400 9150 11400 11300
-Wire Bus Line
-	11600 9950 11600 11100
-Wire Bus Line
-	1600 4100 1600 8250
-Wire Bus Line
-	5600 5200 5600 7450
-Wire Bus Line
-	8000 12300 8000 14200
-Wire Bus Line
-	11500 5200 11500 7450
-Wire Bus Line
-	5800 12300 5800 14200
-Wire Bus Line
-	16000 14950 16000 18150
-Wire Bus Line
-	5300 9950 5300 15400
-Wire Bus Line
-	4900 9150 4900 16100
-Wire Bus Line
-	2400 12300 2400 14600
-Wire Bus Line
-	9600 6650 9600 10750
-Wire Bus Line
-	7700 9150 7700 10750
-Wire Bus Line
-	4300 6550 4300 12100
-Wire Bus Line
-	13500 8350 13500 11700
-Wire Bus Line
-	8000 5950 8000 9850
-Wire Bus Line
-	14400 14250 14400 17950
 Text Notes 11800 3200 0    50   ~ 0
 Roughly 2.3~~2.4V\nsquare signal output
+$Comp
+L 74xx:74LS125 UP3
+U 5 1 695390A5
+P 10700 21500
+F 0 "UP3" V 10450 21600 50  0000 L CNN
+F 1 "74LS125" V 10950 21450 50  0000 L CNN
+F 2 "Package_SO:SOIC-14_3.9x8.7mm_P1.27mm" H 10700 21500 50  0001 C CNN
+F 3 "http://www.ti.com/lit/gpn/sn74LS126a" H 10700 21500 50  0001 C CNN
+	5    10700 21500
+	0    -1   1    0
+$EndComp
+Wire Bus Line
+	5000 11400 11300 11400
+Wire Bus Line
+	4800 11600 11100 11600
+Wire Bus Line
+	4600 12000 8100 12000
+Wire Bus Line
+	4400 12200 7900 12200
+Wire Bus Line
+	11200 8950 11200 11500
+Wire Wire Line
+	7500 14800 8700 14800
+Wire Wire Line
+	3900 9850 5200 9850
+Wire Bus Line
+	5000 16200 7900 16200
+Wire Wire Line
+	3700 14400 4800 14400
+Wire Wire Line
+	3900 9050 4800 9050
+Wire Wire Line
+	3900 8850 4600 8850
+Wire Bus Line
+	5800 5300 5800 8650
+Wire Bus Line
+	5900 15500 5900 16100
+Wire Bus Line
+	2200 12100 2200 15400
+Wire Bus Line
+	8200 12100 8200 14800
+Wire Bus Line
+	8000 15500 8000 16100
+Wire Bus Line
+	9400 11700 9400 17250
+Wire Bus Line
+	9100 11500 9100 17650
+Wire Bus Line
+	14200 13650 14200 14650
+Wire Bus Line
+	4500 6150 4500 11900
+Wire Bus Line
+	8800 11300 8800 14700
+Wire Bus Line
+	9800 5300 9800 8550
+Wire Bus Line
+	9500 2300 9500 3900
+Wire Bus Line
+	1500 2400 1500 4000
+Wire Bus Line
+	4700 8950 4700 14500
+Wire Bus Line
+	16200 13650 16200 16850
+Wire Bus Line
+	14100 16650 14100 18150
+Wire Bus Line
+	10000 14900 10000 17050
+Wire Bus Line
+	11400 9150 11400 11300
+Wire Bus Line
+	11600 9950 11600 11100
+Wire Bus Line
+	1600 4100 1600 8250
+Wire Bus Line
+	5600 5200 5600 7450
+Wire Bus Line
+	8000 12300 8000 14200
+Wire Bus Line
+	11500 5200 11500 7450
+Wire Bus Line
+	5800 12300 5800 14200
+Wire Bus Line
+	16000 14950 16000 18150
+Wire Bus Line
+	5300 9950 5300 15400
+Wire Bus Line
+	4900 9150 4900 16100
+Wire Bus Line
+	2400 12300 2400 14600
+Wire Bus Line
+	9600 6650 9600 10750
+Wire Bus Line
+	7700 9150 7700 10750
+Wire Bus Line
+	4300 6550 4300 12100
+Wire Bus Line
+	13500 8350 13500 11700
+Wire Bus Line
+	8000 5950 8000 9850
+Wire Bus Line
+	14400 14250 14400 17950
 $EndSCHEMATC

Commit message: Fixed footprints for Reset Button, X2 and UPA1
Parts:
- SW1: footprint Button_Switch_SMD:SW_Push_SPST_NO_Alps_SKRK -> SNES:SW_Push_SPST_NO_Alps_SKRK
- UPA1: footprint Package_LCC:PLCC-20 -> SNES:PLCC-20
- X2: footprint Crystal:Crystal_SMD_HC49-SD -> Crystal:Crystal_HC49-4H_Vertical
Changed lines of the file:
@@
 F 0 "SW1" V 1950 18000 50  0000 R CNN
 F 1 "RESET" V 1650 18100 50  0000 R CNN
-F 2 "Button_Switch_SMD:SW_Push_SPST_NO_Alps_SKRK" H 1800 18000 50  0001 C CNN
+F 2 "SNES:SW_Push_SPST_NO_Alps_SKRK" H 1800 18000 50  0001 C CNN
 F 3 "~" H 1800 18000 50  0001 C CNN
 	1    1800 17800
@@
 F 0 "X2" H 11400 13500 50  0000 C BNN
 F 1 "24.576MHz" H 11400 13400 50  0000 C BNN
-F 2 "Crystal:Crystal_SMD_HC49-SD" H 11400 13300 50  0001 C CNN
+F 2 "Crystal:Crystal_HC49-4H_Vertical" H 11400 13300 50  0001 C CNN
 F 3 "~" H 11400 13300 50  0001 C CNN
 	1    11400 13300
@@
 F 0 "UPA1" H 13050 21050 50  0000 L CNN
 F 1 "16V8" H 13050 19850 50  0000 L CNN
-F 2 "Package_LCC:PLCC-20" H 13400 20450 50  0001 C CNN
+F 2 "SNES:PLCC-20" H 13400 20450 50  0001 C CNN
 F 3 "" H 13400 20450 50  0001 C CNN
 	1    13400 20450

Commit message: Fixed footprints for SRAM chips
Parts:
- U15: footprint Package_SO:SSOP-28_5.3x10.2mm_P0.65mm -> SNES:SOIC-28W_7.5x17.9mm_P1.27mm
- U16, U4, U5: footprint SNES:SSOP-28_5.3x10.2mm_P0.65mm -> SNES:SOIC-28W_7.5x17.9mm_P1.27mm
Changed lines of the file:
@@
 F 0 "U4" H 8550 5650 50  0000 C CNN
 F 1 "SRAM" H 8750 3950 50  0000 C CNN
-F 2 "SNES:SSOP-28_5.3x10.2mm_P0.65mm" H 8750 5550 50  0001 C CNN
-F 3 "" H 8750 5550 50  0001 C CNN
+F 2 "SNES:SOIC-28W_7.5x17.9mm_P1.27mm" H 8750 5550 50  0001 C CNN
+F 3 "https://www.futurlec.com/Datasheet/Memory/62256.pdf" H 8750 5550 50  0001 C CNN
 	1    8750 5650
 	1    0    0    -1
@@
 F 0 "U5" H 8550 8150 50  0000 C CNN
 F 1 "SRAM" H 8750 6450 50  0000 C CNN
-F 2 "SNES:SSOP-28_5.3x10.2mm_P0.65mm" H 8750 8050 50  0001 C CNN
-F 3 "" H 8750 8050 50  0001 C CNN
+F 2 "SNES:SOIC-28W_7.5x17.9mm_P1.27mm" H 8750 8050 50  0001 C CNN
+F 3 "https://www.futurlec.com/Datasheet/Memory/62256.pdf" H 8750 8050 50  0001 C CNN
 	1    8750 8150
 	1    0    0    -1
@@
 F 0 "U16" H 15000 16250 50  0000 L CNN
 F 1 "PSRAM" H 15250 14550 50  0000 C CNN
-F 2 "SNES:SSOP-28_5.3x10.2mm_P0.65mm" H 15250 16150 50  0001 C CNN
-F 3 "" H 15250 16150 50  0001 C CNN
+F 2 "SNES:SOIC-28W_7.5x17.9mm_P1.27mm" H 15250 16150 50  0001 C CNN
+F 3 "https://wakamatsu.co.jp/waka/LH5P832-10_to_LH5P832N-12%20(2).pdf" H 15250 16150 50  0001 C CNN
 	1    15250 16250
 	1    0    0    -1
@@
 F 0 "U15" H 15000 13950 50  0000 L CNN
 F 1 "PSRAM" H 15250 12250 50  0000 C CNN
-F 2 "Package_SO:SSOP-28_5.3x10.2mm_P0.65mm" H 15250 13850 50  0001 C CNN
-F 3 "" H 15250 13850 50  0001 C CNN
+F 2 "SNES:SOIC-28W_7.5x17.9mm_P1.27mm" H 15250 13850 50  0001 C CNN
+F 3 "https://wakamatsu.co.jp/waka/LH5P832-10_to_LH5P832N-12%20(2).pdf" H 15250 13850 50  0001 C CNN
 	1    15250 13950
 	1    0    0    -1

Commit message: Fixed footprint size for C62, rewired RN7882 for better fit on PCB
Parts:
- C62: footprint Capacitor_SMD:CP_Elec_6.3x5.4 -> Capacitor_SMD:CP_Elec_4x5.4
Changed lines of the file:
@@
 NoConn ~ 2300 2200
 NoConn ~ 2300 1800
-Wire Wire Line
-	2000 2200 2000 2300
-Wire Wire Line
-	2200 2500 2200 2200
-Wire Wire Line
-	2100 2400 2100 2200
 Wire Bus Line
 	1500 4000 1600 4100
@@
 Entry Wire Line
 	1500 2700 1600 2600
-Wire Wire Line
-	1600 2300 2000 2300
-Connection ~ 2000 2300
-Wire Wire Line
-	1600 2400 2100 2400
-Connection ~ 2100 2400
-Wire Wire Line
-	1600 2500 2200 2500
-Connection ~ 2200 2500
 Text Label 1600 2300 0    50   ~ 0
 JPIO7
@@
 Text Label 1800 8350 0    50   ~ 0
 JPSTR
-Wire Wire Line
-	2100 2400 3300 2400
 $Comp
 L Diode:BAT54C DA10
@@
 	1600 2600 4300 2600
 Wire Wire Line
-	2200 2500 3800 2500
-Wire Wire Line
 	3300 2200 3300 2400
 Connection ~ 3300 2400
@@
 	7600 2300 7400 2300
 Wire Wire Line
-	2000 2300 2800 2300
-Wire Wire Line
 	2800 2200 2800 2300
 Connection ~ 2800 2300
@@
 F 0 "C62" H 2350 17600 50  0000 L CNN
 F 1 "2.2uF" H 2350 17400 50  0000 L CNN
-F 2 "Capacitor_SMD:CP_Elec_6.3x5.4" H 2300 17500 50  0001 C CNN
+F 2 "Capacitor_SMD:CP_Elec_4x5.4" H 2300 17500 50  0001 C CNN
 F 3 "~" H 2300 17500 50  0001 C CNN
 	1    2300 17500
@@
 	0    -1   1    0
 $EndComp
+Wire Wire Line
+	1600 2500 2000 2500
+Wire Wire Line
+	2100 2400 3300 2400
+Wire Wire Line
+	1600 2400 2100 2400
+Connection ~ 2100 2400
+Wire Wire Line
+	2100 2400 2100 2200
+Wire Wire Line
+	1600 2300 2200 2300
+Wire Wire Line
+	2000 2200 2000 2500
+Connection ~ 2000 2500
+Wire Wire Line
+	2000 2500 3800 2500
+Wire Wire Line
+	2200 2200 2200 2300
 Wire Bus Line
 	5000 11400 11300 11400
@@
 Wire Bus Line
 	14400 14250 14400 17950
+Connection ~ 2200 2300
+Wire Wire Line
+	2200 2300 2800 2300
 $EndSCHEMATC

Commit message: Replaced footprint with 2.54mm pitch for easier routing and debugging
Parts:
- J5, P4: footprint Connector_PinHeader_1.27mm:PinHeader_2x04_P1.27mm_Vertical -> Connector_PinHeader_2.54mm:PinHeader_2x04_P2.54mm_Vertical
Changed lines of the file:
@@
 F 0 "J5" H 19000 8750 50  0000 C CNN
 F 1 "Audio Out Port" H 19000 8250 50  0000 C CNN
-F 2 "Connector_PinHeader_1.27mm:PinHeader_2x04_P1.27mm_Vertical" H 18950 8550 50  0001 C CNN
+F 2 "Connector_PinHeader_2.54mm:PinHeader_2x04_P2.54mm_Vertical" H 18950 8550 50  0001 C CNN
 F 3 "~" H 18950 8550 50  0001 C CNN
 	1    18950 8550
@@
 F 0 "P4" H 19100 7350 50  0000 C CNN
 F 1 "Multi AV Out" H 19100 6850 50  0000 C CNN
-F 2 "Connector_PinHeader_1.27mm:PinHeader_2x04_P1.27mm_Vertical" H 19050 7150 50  0001 C CNN
+F 2 "Connector_PinHeader_2.54mm:PinHeader_2x04_P2.54mm_Vertical" H 19050 7150 50  0001 C CNN
 F 3 "~" H 19050 7150 50  0001 C CNN
 	1    19050 7150
@@
 Wire Wire Line
 	2200 2200 2200 2300
+Connection ~ 2200 2300
+Wire Wire Line
+	2200 2300 2800 2300
 Wire Bus Line
 	5000 11400 11300 11400
@@
 Wire Bus Line
 	14400 14250 14400 17950
-Connection ~ 2200 2300
-Wire Wire Line
-	2200 2300 2800 2300
 $EndSCHEMATC
